File: PWMWatch/PWMWatch.kicad_pcb (KiCad board)
At the start: 2 copper layers, 70 parts, among them J1 USB_C_Receptacle_USB2.0_14P, J2 5025700893, Q1 PMOS, SW1 RST, SW2 BOOT, SW3 SW_Push, U1 STM32WB50CGUx, U2 AP3012, U3 TVS1400DRV, U6 NCP1117-3.3_SOT223

Commit message: placements + fixed all the wrong footprints
Parts:
- added R14: 5.1k, Resistor_SMD:R_0603_1608Metric, B.Cu at (229.2, 118.5)
- added R15: 5.1k, Resistor_SMD:R_0603_1608Metric, B.Cu at (229.2, 115.5)
- BT1, C10, C11, C12, C15, C21, C27, C3, C4, C5, C6, C7, C8, C9, D4, D5, J2, MCP1, Q1, R10, R12, R26, R27, R28, R29, R30, R5, R6, R7, R8, R9: moved to B.Cu
- moved C14 302.2 mm to (231.6, 107.9), turned to -90 degrees
- moved C21 299.5 mm to (228.9, 122.8)
- moved C4 296.5 mm to (217.1, 116.7), turned to -45 degrees
- moved C5 294.4 mm to (214.9, 117.5), turned to -45 degrees
- moved C6 292.6 mm to (213.2, 121.6), turned to 45 degrees
- moved C27 292.5 mm to (230.4, 128.8)
- moved C7 292.3 mm to (212.7, 119.2), turned to 45 degrees
- moved D5 291.5 mm to (229.5, 125.0), turned to 180 degrees
- moved J1 291.2 mm to (229.9, 116.0), turned to 90 degrees
- moved SW2 290.7 mm to (227.7, 107.8), turned to 180 degrees
- moved C3 289.1 mm to (209.6, 116.2), turned to -135 degrees
- moved C8 288.5 mm to (213.5, 114.9), turned to 45 degrees
- moved C2 288.5 mm to (208.9, 107.3), turned to -90 degrees
- moved BT1 287.9 mm to (217.9, 128.0)
- moved C9 287.3 mm to (212.3, 112.0), turned to 135 degrees
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Connections:
- J1 pad A5: unconnected-(J1-CC1-PadA5) -> Net-(J1-CC1)
- J1 pad B5: unconnected-(J1-CC2-PadB5) -> Net-(J1-CC2)
Routing:
- net /V_{BUS}: track 0.00 -> 7.96 mm
- net Net-(J1-CC2): track 0.00 -> 3.22 mm, vias 0 -> 1
- net Net-(J1-CC1): track 0.00 -> 3.15 mm, vias 0 -> 1
- net /D-: track 0.00 -> 2.50 mm
- net /D+: track 0.00 -> 2.50 mm
Other:
- board outline added: 45 x 33.5 mm
- rule pad_to_mask_clearance: 0 -> 0.1

Commit message: pcb done 4th time
Parts:
- added R16: 10k, Resistor_SMD:R_0603_1608Metric, F.Cu at (107.8, 98.0)
- added R17: 10k, Resistor_SMD:R_0603_1608Metric, F.Cu at (112.3, 98.5)
- added R18: 10k, Resistor_SMD:R_0603_1608Metric, F.Cu at (107.4, 91.6)
- BT1: footprint Connector_JST:JST_PH_B2B-PH-K_1x02_P2.00mm_Vertical -> Watch:CONN_BM02B-SRSS-TB_JST
- C10, C11, C12, C15, C21, C27, C3, C4, C5, C6, C7, C8, C9, D4, D5, MCP1, Q1, R10, R14, R15, R26, R27, R28, R29, R5, R6, R8: moved to F.Cu
- C18, C19, C2, C20, C22, D2, L2, R11, U6: moved to B.Cu
- moved C14 122.8 mm to (110.1, 89.7), turned to 90 degrees
- moved SW2 114.3 mm to (114.6, 90.8), turned to -90 degrees
- moved R2 113.5 mm to (112.0, 89.5), turned to -90 degrees
- moved C1 112.5 mm to (111.6, 83.9), turned to 90 degrees
- moved D5 103.3 mm to (127.7, 107.2), turned to 0 degrees
- moved C4 101.8 mm to (118.2, 92.7), turned to 0 degrees
- moved C27 101.5 mm to (132.1, 103.7), turned to 180 degrees
- moved C5 101.0 mm to (116.5, 94.8), turned to 0 degrees
- moved R28 101.0 mm to (132.1, 105.2), turned to 180 degrees
- moved R10 99.8 mm to (118.4, 88.1), turned to -90 degrees
- moved C6 99.7 mm to (116.4, 97.6), turned to 0 degrees
- moved R12 99.3 mm to (118.4, 88.1), turned to -90 degrees
- moved R27 99.0 mm to (134.4, 106.6), turned to -90 degrees
- moved Q1 98.2 mm to (128.8, 103.6), turned to -90 degrees
- moved C21 98.2 mm to (131.9, 107.2), turned to 180 degrees
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Connections:
- U1 pad 13: unconnected-(U1-PA4-Pad13) -> /BTN
- U1 pad 14: /BTN -> /SCK
- U1 pad 15: unconnected-(U1-PA6-Pad15) -> /MISO
- U1 pad 16: unconnected-(U1-PA7-Pad16) -> /MOSI
Routing:
- net +3V3: track 0.00 -> 176.3 mm, vias 0 -> 10
- net /SCL: track 0.00 -> 58.1 mm, vias 0 -> 7
- net Net-(U1-VBAT): track 0.00 -> 57.9 mm, vias 0 -> 2
- net /SDA: track 0.00 -> 51.6 mm, vias 0 -> 6
- net /MOSI: track 0.00 -> 37.3 mm, vias 0 -> 2
- net /BTN: track 0.00 -> 27.1 mm, vias 0 -> 2
- net /V_{BUS}: track 7.96 -> 34.8 mm
- net Net-(U1-NRST): track 0.00 -> 24.9 mm, vias 0 -> 2
- net /V_{Li}: track 0.00 -> 23.0 mm, vias 0 -> 3
- net /VOLED: track 0.00 -> 20.9 mm
- net /V_{BAT}: track 0.00 -> 20.4 mm, vias 0 -> 2
- net Net-(U1-PH3): track 0.00 -> 20.1 mm, vias 0 -> 2
- net /MISO: track 0.00 -> 17.7 mm, vias 0 -> 2
- net /SCK: track 0.00 -> 15.8 mm, vias 0 -> 2
- net GND: track 0.00 -> 13.8 mm, vias 0 -> 21
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- added copper zone on B.Cu, net GND
- added copper zone on F.Cu, net GND
Other:
- board size 45 x 33.5 mm -> 45 x 30 mm
- board text added: "asadpetwalker '27"

Commit message: all the stuff done
Parts:
- added REF**: MountingHole_2.2mm_M2, MountingHole:MountingHole_2.2mm_M2, F.Cu at (142.8, 84.1)
- added REF**: MountingHole_2.2mm_M2, MountingHole:MountingHole_2.2mm_M2, F.Cu at (103.6, 108.3)
- CC1: footprint Watch:BAT_BK-414 -> Watch:BAT_2994
- moved R1 1.20 mm to (114.8, 101.4), turned to 90 degrees
- moved C13 0.53 mm to (114.9, 104.0)
- moved CC1 0.30 mm to (110.5, 107.8)
Routing:
- net +3V3: track 176.3 -> 177.2 mm
- net GND: vias 21 -> 22
Other:
- rule pad_to_mask_clearance: 0.1 -> 0
